File: jbox_kicad.sch (KiCad schematic (older format))
At the start: 11 parts, among them U1 LM2596HVS, U2 DS18B20, U3 mini_esp32

Commit message: 2nd version
Connections:
- net GND: no longer BT1.1 (+), C1.1, C2.1, R2.1, U1.1 (Vin), U1.2 (Vout), U3.36 (IO_02)
- new net VDD41: BT1.1 (+), U1.1 (Vin)
- new net VDD5: C1.1, C2.1, R2.1, U1.2 (Vout), U3.36 (IO_02)
Other:
- moved on the sheet: C1, C2, R2, R3
Changed lines of the file:
@@
 	1100 1100 1700 1100
-Wire Wire Line
-	1100 1500 1100 1700
-Wire Wire Line
-	1100 1700 1700 1700
 Wire Wire Line
 	2800 2950 2800 3350
@@
 NoConn ~ 5600 1350
 NoConn ~ 5600 1150
-Wire Wire Line
-	1700 1700 1700 1100
 $Comp
 L power:GND #PWR01
 U 1 1 6090D592
-P 1700 1700
-F 0 "#PWR01" H 1700 1450 50  0001 C CNN
-F 1 "GND" H 1705 1527 50  0000 C CNN
-F 2 "" H 1700 1700 50  0001 C CNN
-F 3 "" H 1700 1700 50  0001 C CNN
-	1    1700 1700
-	1    0    0    -1
-$EndComp
-Connection ~ 1700 1700
+P 1100 1500
+F 0 "#PWR01" H 1100 1250 50  0001 C CNN
+F 1 "GND" H 1105 1327 50  0000 C CNN
+F 2 "" H 1100 1500 50  0001 C CNN
+F 3 "" H 1100 1500 50  0001 C CNN
+	1    1100 1500
+	1    0    0    -1
+$EndComp
 $Comp
 L power:GND #PWR0101
@@
 Text GLabel 1450 4500 1    50   Input ~ 0
 VDD33
-Text Label 4300 4300 0    50   ~ 0
+Text Label 4100 4200 0    50   ~ 0
 VoltageDivider
-Text GLabel 4400 4650 0    50   Input ~ 0
+Text GLabel 4200 4350 0    50   Input ~ 0
 VDD5
 Wire Wire Line
-	4400 5450 5050 5450
-Wire Wire Line
-	5050 5450 5050 5350
-Wire Wire Line
-	5050 4450 4400 4450
-Wire Wire Line
-	4400 4450 4400 5450
+	4850 5350 4850 5250
+Wire Wire Line
+	4850 4350 4200 4350
 $Comp
 L Device:R R2
 U 1 1 609485CD
-P 5050 4700
-F 0 "R2" H 5120 4746 50  0000 L CNN
-F 1 "1000" H 5120 4655 50  0000 L CNN
-F 2 "Resistor_THT:R_Axial_DIN0207_L6.3mm_D2.5mm_P10.16mm_Horizontal" V 4980 4700 50  0001 C CNN
-F 3 "~" H 5050 4700 50  0001 C CNN
-	1    5050 4700
+P 4850 4600
+F 0 "R2" H 4920 4646 50  0000 L CNN
+F 1 "1000" H 4920 4555 50  0000 L CNN
+F 2 "Resistor_THT:R_Axial_DIN0207_L6.3mm_D2.5mm_P10.16mm_Horizontal" V 4780 4600 50  0001 C CNN
+F 3 "~" H 4850 4600 50  0001 C CNN
+	1    4850 4600
 	1    0    0    -1
 $EndComp
@@
 L Device:R R3
 U 1 1 60948C85
-P 5050 5200
-F 0 "R3" H 5120 5246 50  0000 L CNN
-F 1 "2000" H 5120 5155 50  0000 L CNN
-F 2 "Resistor_THT:R_Axial_DIN0207_L6.3mm_D2.5mm_P10.16mm_Horizontal" V 4980 5200 50  0001 C CNN
-F 3 "~" H 5050 5200 50  0001 C CNN
-	1    5050 5200
+P 4850 5100
+F 0 "R3" H 4920 5146 50  0000 L CNN
+F 1 "2000" H 4920 5055 50  0000 L CNN
+F 2 "Resistor_THT:R_Axial_DIN0207_L6.3mm_D2.5mm_P10.16mm_Horizontal" V 4780 5100 50  0001 C CNN
+F 3 "~" H 4850 5100 50  0001 C CNN
+	1    4850 5100
 	1    0    0    -1
 $EndComp
@@
 L power:GND #PWR0105
 U 1 1 609491C1
-P 5050 5450
-F 0 "#PWR0105" H 5050 5200 50  0001 C CNN
-F 1 "GND" H 5055 5277 50  0000 C CNN
-F 2 "" H 5050 5450 50  0001 C CNN
-F 3 "" H 5050 5450 50  0001 C CNN
-	1    5050 5450
-	1    0    0    -1
-$EndComp
-Connection ~ 5050 5450
-Text GLabel 5050 5000 2    50   Input ~ 0
+P 4850 5350
+F 0 "#PWR0105" H 4850 5100 50  0001 C CNN
+F 1 "GND" H 4855 5177 50  0000 C CNN
+F 2 "" H 4850 5350 50  0001 C CNN
+F 3 "" H 4850 5350 50  0001 C CNN
+	1    4850 5350
+	1    0    0    -1
+$EndComp
+Text GLabel 4850 4900 2    50   Input ~ 0
 VDD33
 Text Label 5250 1250 1    50   ~ 0
@@
 Text GLabel 3200 2750 2    50   Input ~ 0
 VDD5
-Wire Wire Line
-	4900 1250 4550 1250
-Wire Wire Line
-	5600 1250 4900 1250
-Connection ~ 4900 1250
-$Comp
-L power:GND #PWR0102
-U 1 1 60956816
-P 4650 1600
-F 0 "#PWR0102" H 4650 1350 50  0001 C CNN
-F 1 "GND" H 4655 1427 50  0000 C CNN
-F 2 "" H 4650 1600 50  0001 C CNN
-F 3 "" H 4650 1600 50  0001 C CNN
-	1    4650 1600
-	1    0    0    -1
-$EndComp
-$Comp
-L Device:C C1
-U 1 1 6095681C
-P 4650 1450
-F 0 "C1" H 4765 1496 50  0000 L CNN
-F 1 "100uF" H 4765 1405 50  0000 L CNN
-F 2 "Capacitor_THT:C_Axial_L5.1mm_D3.1mm_P7.50mm_Horizontal" H 4688 1300 50  0001 C CNN
-F 3 "~" H 4650 1450 50  0001 C CNN
-	1    4650 1450
-	1    0    0    -1
-$EndComp
-Text Label 4650 1600 0    50   ~ 0
-GND
-$Comp
-L power:GND #PWR0103
-U 1 1 60956823
-P 5100 1600
-F 0 "#PWR0103" H 5100 1350 50  0001 C CNN
-F 1 "GND" H 5105 1427 50  0000 C CNN
-F 2 "" H 5100 1600 50  0001 C CNN
-F 3 "" H 5100 1600 50  0001 C CNN
-	1    5100 1600
-	1    0    0    -1
-$EndComp
-$Comp
-L Device:C C2
-U 1 1 60956829
-P 5100 1450
-F 0 "C2" H 5215 1496 50  0000 L CNN
-F 1 "10uF" H 5215 1405 50  0000 L CNN
-F 2 "Capacitor_THT:C_Axial_L5.1mm_D3.1mm_P7.50mm_Horizontal" H 5138 1300 50  0001 C CNN
-F 3 "~" H 5100 1450 50  0001 C CNN
-	1    5100 1450
-	1    0    0    -1
-$EndComp
-Text Label 5100 1600 0    50   ~ 0
-GND
-Wire Wire Line
-	4900 1250 4900 1300
-Wire Wire Line
-	4900 1300 4650 1300
-Wire Wire Line
-	4900 1300 5100 1300
-Connection ~ 4900 1300
-Text Label 5050 4950 2    50   ~ 0
+Text Label 4850 4850 2    50   ~ 0
 VDD5toVDD33
 Wire Wire Line
-	5050 4850 5050 5050
-Text Label 4550 4450 0    50   ~ 0
+	4850 4750 4850 4950
+Text Label 4350 4350 0    50   ~ 0
 VDD5toR1
-Text Label 4550 5450 0    50   ~ 0
+Text Label 4850 5350 0    50   ~ 0
 VDD5toR2
 Wire Wire Line
-	5050 4550 5050 4450
+	4850 4450 4850 4350
 NoConn ~ 5600 2050
 NoConn ~ 5600 2750
 Text Label 5500 3450 1    50   ~ 0
 DStoESP
+Text Label 5150 1550 0    50   ~ 0
+GND
+$Comp
+L Device:C C2
+U 1 1 60956829
+P 5150 1400
+F 0 "C2" H 5265 1446 50  0000 L CNN
+F 1 "10uF" H 5265 1355 50  0000 L CNN
+F 2 "Capacitor_THT:C_Axial_L5.1mm_D3.1mm_P7.50mm_Horizontal" H 5188 1250 50  0001 C CNN
+F 3 "~" H 5150 1400 50  0001 C CNN
+	1    5150 1400
+	1    0    0    -1
+$EndComp
+$Comp
+L power:GND #PWR0103
+U 1 1 60956823
+P 5150 1550
+F 0 "#PWR0103" H 5150 1300 50  0001 C CNN
+F 1 "GND" H 5155 1377 50  0000 C CNN
+F 2 "" H 5150 1550 50  0001 C CNN
+F 3 "" H 5150 1550 50  0001 C CNN
+	1    5150 1550
+	1    0    0    -1
+$EndComp
+Text Label 4700 1550 0    50   ~ 0
+GND
+$Comp
+L Device:C C1
+U 1 1 6095681C
+P 4700 1400
+F 0 "C1" H 4815 1446 50  0000 L CNN
+F 1 "100uF" H 4815 1355 50  0000 L CNN
+F 2 "Capacitor_THT:C_Axial_L5.1mm_D3.1mm_P7.50mm_Horizontal" H 4738 1250 50  0001 C CNN
+F 3 "~" H 4700 1400 50  0001 C CNN
+	1    4700 1400
+	1    0    0    -1
+$EndComp
+$Comp
+L power:GND #PWR0102
+U 1 1 60956816
+P 4700 1550
+F 0 "#PWR0102" H 4700 1300 50  0001 C CNN
+F 1 "GND" H 4705 1377 50  0000 C CNN
+F 2 "" H 4700 1550 50  0001 C CNN
+F 3 "" H 4700 1550 50  0001 C CNN
+	1    4700 1550
+	1    0    0    -1
+$EndComp
+Wire Wire Line
+	4550 1250 4700 1250
+Connection ~ 4700 1250
+Wire Wire Line
+	4700 1250 5150 1250
+Connection ~ 5150 1250
+Wire Wire Line
+	5150 1250 5600 1250
 $EndSCHEMATC
